File: Kurupira Arthur.sch (KiCad schematic (older format))
At the start: 14 parts

Commit message: Testando no pc o novo email
Parts:
- added R?: R, symbol Device:R
- D?: symbol LED -> Kurupira-Arthur-rescue:LED
- J?: symbol Raspberry_Pi_2_3 -> Kurupira-Arthur-rescue:Raspberry_Pi_2_3
- PIR?: symbol PIR_Motion_Sensor -> Kurupira-Arthur-rescue:PIR_Motion_Sensor
- Q?: symbol Q_NPN_BCE -> Kurupira-Arthur-rescue:Q_NPN_BCE
- R? (x7): symbol R -> Kurupira-Arthur-rescue:R
- TH?: symbol DHT11_Temperature_Humidity -> Kurupira-Arthur-rescue:DHT11_Temperature_Humidity
- U?: symbol YL-38 -> Kurupira-Arthur-rescue:YL-38
- U?: symbol FC-37 -> Kurupira-Arthur-rescue:FC-37
Other:
- note added: "TEXTO PARA TESTAR O GIT HUB\n"
Changed lines of the file:
@@
-EESchema Schematic File Version 2
-LIBS:power
-LIBS:device
-LIBS:switches
-LIBS:relays
-LIBS:motors
-LIBS:transistors
-LIBS:conn
-LIBS:linear
-LIBS:regul
-LIBS:74xx
-LIBS:cmos4000
-LIBS:adc-dac
-LIBS:memory
-LIBS:xilinx
-LIBS:microcontrollers
-LIBS:dsp
-LIBS:microchip
-LIBS:analog_switches
-LIBS:motorola
-LIBS:texas
-LIBS:intel
-LIBS:audio
-LIBS:interface
-LIBS:digital-audio
-LIBS:philips
-LIBS:display
-LIBS:A6_GSM
-LIBS:misc
-LIBS:nodemcu
-LIBS:sensors (2)
-LIBS:cypress
-LIBS:siliconi
-LIBS:opto
-LIBS:atmel
-LIBS:contrib
-LIBS:valves
-LIBS:yl-38
+EESchema Schematic File Version 4
 LIBS:Kurupira Arthur-cache
-EELAYER 25 0
+EELAYER 26 0
 EELAYER END
 $Descr A4 11693 8268
@@
 $EndDescr
 $Comp
-L PIR_Motion_Sensor PIR?
+L Kurupira-Arthur-rescue:PIR_Motion_Sensor PIR?
 U 1 1 5AB500A8
 P 7300 1500
@@
 $EndComp
 $Comp
-L Raspberry_Pi_2_3 J?
+L Kurupira-Arthur-rescue:Raspberry_Pi_2_3 J?
 U 1 1 5AB5011B
 P 5300 3550
@@
 $EndComp
 $Comp
-L DHT11_Temperature_Humidity TH?
+L Kurupira-Arthur-rescue:DHT11_Temperature_Humidity TH?
 U 1 1 5AB502A0
 P 10050 1900
@@
 $EndComp
 $Comp
-L Q_NPN_BCE Q?
+L Kurupira-Arthur-rescue:Q_NPN_BCE Q?
 U 1 1 5AB502D9
 P 8950 2900
@@
 $EndComp
 $Comp
-L R R?
+L Kurupira-Arthur-rescue:R R?
 U 1 1 5AB50322
 P 9050 2350
@@
 $EndComp
 $Comp
-L R R?
+L Kurupira-Arthur-rescue:R R?
 U 1 1 5AB5035D
 P 8600 2900
@@
 $EndComp
 Wire Wire Line
-	9050 2500 9050 2700
-$Comp
-L GND #PWR?
+	9050 2500 9050 2600
+$Comp
+L power:GND #PWR?
 U 1 1 5AD0AD1B
 P 9050 3250
@@
 	9050 2000 9050 2200
 $Comp
-L +3.3V #PWR?
+L power:+3.3V #PWR?
 U 1 1 5AD0B1EA
 P 9050 2000
@@
 $EndComp
 $Comp
-L +3.3V #PWR?
+L power:+3.3V #PWR?
 U 1 1 5AD0B2C6
 P 7200 1400
@@
 	7200 1400 7200 1500
 $Comp
-L GND #PWR?
+L power:GND #PWR?
 U 1 1 5AD0B2F8
 P 7400 1400
@@
 PIR
 Wire Wire Line
-	7300 1100 7300 1500
+	7300 1100 7300 1150
 Text GLabel 9450 2600 2    60   Output ~ 0
 RPi5
@@
 RPi11
 Wire Wire Line
-	7900 1150 7300 1150
+	7900 1150 7450 1150
 Connection ~ 7300 1150
 Text GLabel 9950 2550 3    60   Output ~ 0
 RPi22
 Wire Wire Line
-	10050 1900 10050 2000
-$Comp
-L GND #PWR?
+	10050 1900 10050 1950
+$Comp
+L power:GND #PWR?
 U 1 1 5AD0BDB1
 P 10150 2300
@@
 As labels GPIO2 e GPIO4 podem ser quaisquer GPIO da RSP.\nElas não podem ser apenas GPIO3.
 $Comp
-L YL-38 U?
+L Kurupira-Arthur-rescue:YL-38 U?
 U 1 1 5B7B1847
 P 8100 4300
@@
 	8650 4100 8550 4100
 $Comp
-L +5V #PWR?
+L power:+5V #PWR?
 U 1 1 5B7B1B97
 P 8650 3800
@@
 $EndComp
 $Comp
-L GND #PWR?
+L power:GND #PWR?
 U 1 1 5B7B1BBE
 P 8650 4700
@@
 	8550 4200 8650 4200
 Wire Wire Line
-	8650 4200 8650 4700
-$Comp
-L R R?
+	8650 4200 8650 4600
+$Comp
+L Kurupira-Arthur-rescue:R R?
 U 1 1 5B7B1C01
 P 9150 4150
@@
 $EndComp
 $Comp
-L R R?
+L Kurupira-Arthur-rescue:R R?
 U 1 1 5B7B1C61
 P 9150 4450
@@
 $EndComp
 $Comp
-L R R?
+L Kurupira-Arthur-rescue:R R?
 U 1 1 5B7B1CD8
 P 9150 4750
@@
 	4250 3050 4400 3050
 $Comp
-L FC-37 U?
+L Kurupira-Arthur-rescue:FC-37 U?
 U 1 1 5B7B2991
 P 7100 4300
@@
 	4200 3800 4100 3800
 $Comp
-L +5V #PWR?
+L power:+5V #PWR?
 U 1 1 5B7B2F4D
 P 10050 2000
@@
 $EndComp
 $Comp
-L R R?
+L Kurupira-Arthur-rescue:R R?
 U 1 1 5B7B2F77
 P 9950 2050
@@
 	9950 2200 9950 2550
 $Comp
-L LED D?
+L Kurupira-Arthur-rescue:LED D?
 U 1 1 5B7B3797
 P 7600 750
@@
 $EndComp
 $Comp
-L R R?
+L Kurupira-Arthur-rescue:R R?
 U 1 1 5B7B37F2
 P 7900 750
@@
 	8050 1500 7400 1500
 Connection ~ 7400 1500
+Wire Wire Line
+	9050 2600 9050 2700
+Wire Wire Line
+	7300 1150 7300 1500
+Wire Wire Line
+	8650 4600 8650 4700
+Wire Wire Line
+	10050 1950 10050 2000
+Wire Wire Line
+	7450 1150 7300 1150
+$Comp
+L Device:R R?
+U 1 1 5B93C45B
+P 2450 5600
+F 0 "R?" H 2520 5646 50  0000 L CNN
+F 1 "R" H 2520 5555 50  0000 L CNN
+F 2 "" V 2380 5600 50  0001 C CNN
+F 3 "~" H 2450 5600 50  0001 C CNN
+	1    2450 5600
+	1    0    0    -1
+$EndComp
+Text Notes 1950 5100 0    60   ~ 0
+TEXTO PARA TESTAR O GIT HUB\n
 $EndSCHEMATC

Commit message: atualizando o email
Connections:
- net labels added: VCC
Changed lines of the file:
@@
 Text Notes 1950 5100 0    60   ~ 0
 TEXTO PARA TESTAR O GIT HUB\n
+$Comp
+L power:VCC #PWR?
+U 1 1 5B93C5C0
+P 2450 5400
+F 0 "#PWR?" H 2450 5250 50  0001 C CNN
+F 1 "VCC" H 2467 5573 50  0000 C CNN
+F 2 "" H 2450 5400 50  0001 C CNN
+F 3 "" H 2450 5400 50  0001 C CNN
+	1    2450 5400
+	1    0    0    -1
+$EndComp
 $EndSCHEMATC

Commit message: upando o mais atual
Parts:
- removed R?: R, symbol Device:R
- added Q?: BS108, TO_SOT_Packages_THT:TO-92_Molded_Narrow, symbol BS108
- added R? (x2): R, symbol R
- added RV?: POT, symbol POT
- added U?: LM324, symbol LM324
- D?: symbol Kurupira-Arthur-rescue:LED -> LED
- J?: symbol Kurupira-Arthur-rescue:Raspberry_Pi_2_3 -> Raspberry_Pi_2_3
- PIR?: symbol Kurupira-Arthur-rescue:PIR_Motion_Sensor -> PIR_Motion_Sensor
- Q?: symbol Kurupira-Arthur-rescue:Q_NPN_BCE -> Q_NPN_BCE
- R? (x7): symbol Kurupira-Arthur-rescue:R -> R
- TH?: symbol Kurupira-Arthur-rescue:DHT11_Temperature_Humidity -> DHT11_Temperature_Humidity
- U?: symbol Kurupira-Arthur-rescue:YL-38 -> YL-38
- U?: symbol Kurupira-Arthur-rescue:FC-37 -> FC-37
Connections:
- net labels added: VBatt
- net labels removed: VCC
- wire segments 44 -> 58
Other:
- note added: "Parte que desliga a raspberry depois de uma tensão."
- note removed: "TEXTO PARA TESTAR O GIT HUB\n"

Commit message: aberto dps de upado
Parts:
- D?: symbol LED -> Kurupira-Arthur-rescue:LED
- J?: symbol Raspberry_Pi_2_3 -> Kurupira-Arthur-rescue:Raspberry_Pi_2_3
- PIR?: symbol PIR_Motion_Sensor -> Kurupira-Arthur-rescue:PIR_Motion_Sensor
- Q?: symbol Q_NPN_BCE -> Kurupira-Arthur-rescue:Q_NPN_BCE
- Q?: symbol BS108 -> Kurupira-Arthur-rescue:BS108
- R? (x9): symbol R -> Kurupira-Arthur-rescue:R
- RV?: symbol POT -> Kurupira-Arthur-rescue:POT
- TH?: symbol DHT11_Temperature_Humidity -> Kurupira-Arthur-rescue:DHT11_Temperature_Humidity
- U?: symbol YL-38 -> Kurupira-Arthur-rescue:YL-38
- U?: symbol FC-37 -> Kurupira-Arthur-rescue:FC-37
- U?: symbol LM324 -> Kurupira-Arthur-rescue:LM324
Changed lines of the file:
@@
-EESchema Schematic File Version 2
-LIBS:power
-LIBS:device
-LIBS:switches
-LIBS:relays
-LIBS:motors
-LIBS:transistors
-LIBS:conn
-LIBS:linear
-LIBS:regul
-LIBS:74xx
-LIBS:cmos4000
-LIBS:adc-dac
-LIBS:memory
-LIBS:xilinx
-LIBS:microcontrollers
-LIBS:dsp
-LIBS:microchip
-LIBS:analog_switches
-LIBS:motorola
-LIBS:texas
-LIBS:intel
-LIBS:audio
-LIBS:interface
-LIBS:digital-audio
-LIBS:philips
-LIBS:display
-LIBS:A6_GSM
-LIBS:misc
-LIBS:nodemcu
-LIBS:sensors (2)
-LIBS:cypress
-LIBS:siliconi
-LIBS:opto
-LIBS:atmel
-LIBS:contrib
-LIBS:valves
-LIBS:yl-38
-LIBS:fc-37
+EESchema Schematic File Version 4
 LIBS:Kurupira Arthur-cache
-EELAYER 25 0
+EELAYER 26 0
 EELAYER END
 $Descr A4 11693 8268
@@
 $EndDescr
 $Comp
-L PIR_Motion_Sensor PIR?
+L Kurupira-Arthur-rescue:PIR_Motion_Sensor PIR?
 U 1 1 5AB500A8
 P 7300 1500
@@
 $EndComp
 $Comp
-L Raspberry_Pi_2_3 J?
+L Kurupira-Arthur-rescue:Raspberry_Pi_2_3 J?
 U 1 1 5AB5011B
 P 5300 3550
@@
 $EndComp
 $Comp
-L DHT11_Temperature_Humidity TH?
+L Kurupira-Arthur-rescue:DHT11_Temperature_Humidity TH?
 U 1 1 5AB502A0
 P 10050 1900
@@
 $EndComp
 $Comp
-L Q_NPN_BCE Q?
+L Kurupira-Arthur-rescue:Q_NPN_BCE Q?
 U 1 1 5AB502D9
 P 8950 2900
@@
 $EndComp
 $Comp
-L R R?
+L Kurupira-Arthur-rescue:R R?
 U 1 1 5AB50322
 P 9050 2350
@@
 $EndComp
 $Comp
-L R R?
+L Kurupira-Arthur-rescue:R R?
 U 1 1 5AB5035D
 P 8600 2900
@@
 $EndComp
 Wire Wire Line
-	9050 2500 9050 2700
-$Comp
-L GND #PWR?
+	9050 2500 9050 2600
+$Comp
+L power:GND #PWR?
 U 1 1 5AD0AD1B
 P 9050 3250
@@
 	9050 2000 9050 2200
 $Comp
-L +3.3V #PWR?
+L power:+3.3V #PWR?
 U 1 1 5AD0B1EA
 P 9050 2000
@@
 $EndComp
 $Comp
-L +3.3V #PWR?
+L power:+3.3V #PWR?
 U 1 1 5AD0B2C6
 P 7200 1400
@@
 	7200 1400 7200 1500
 $Comp
-L GND #PWR?
+L power:GND #PWR?
 U 1 1 5AD0B2F8
 P 7400 1400
@@
 PIR
 Wire Wire Line
-	7300 1100 7300 1500
+	7300 1100 7300 1150
 Text GLabel 9450 2600 2    60   Output ~ 0
 RPi5
@@
 RPi11
 Wire Wire Line
-	7300 1150 7900 1150
+	7300 1150 7450 1150
 Connection ~ 7300 1150
 Text GLabel 9950 2550 3    60   Output ~ 0
 RPi22
 Wire Wire Line
-	10050 1900 10050 2000
-$Comp
-L GND #PWR?
+	10050 1900 10050 1950
+$Comp
+L power:GND #PWR?
 U 1 1 5AD0BDB1
 P 10150 2300
@@
 As labels GPIO2 e GPIO4 podem ser quaisquer GPIO da RSP.\nElas não podem ser apenas GPIO3.
 $Comp
-L YL-38 U?
+L Kurupira-Arthur-rescue:YL-38 U?
 U 1 1 5B7B1847
 P 8100 4300
@@
 	8650 4100 8550 4100
 $Comp
-L +5V #PWR?
+L power:+5V #PWR?
 U 1 1 5B7B1B97
 P 8650 3800
@@
 $EndComp
 $Comp
-L GND #PWR?
+L power:GND #PWR?
 U 1 1 5B7B1BBE
 P 8650 4700
@@
 	8550 4200 8650 4200
 Wire Wire Line
-	8650 4200 8650 4700
-$Comp
-L R R?
+	8650 4200 8650 4600
+$Comp
+L Kurupira-Arthur-rescue:R R?
 U 1 1 5B7B1C01
 P 9150 4150
@@
 $EndComp
 $Comp
-L R R?
+L Kurupira-Arthur-rescue:R R?
 U 1 1 5B7B1C61
 P 9150 4450
@@
 $EndComp
 $Comp
-L R R?
+L Kurupira-Arthur-rescue:R R?
 U 1 1 5B7B1CD8
 P 9150 4750
@@
 	4250 3050 4400 3050
 $Comp
-L FC-37 U?
+L Kurupira-Arthur-rescue:FC-37 U?
 U 1 1 5B7B2991
 P 7100 4300
@@
 	4200 3800 4100 3800
 $Comp
-L +5V #PWR?
+L power:+5V #PWR?
 U 1 1 5B7B2F4D
 P 10050 2000
@@
 $EndComp
 $Comp
-L R R?
+L Kurupira-Arthur-rescue:R R?
 U 1 1 5B7B2F77
 P 9950 2050
@@
 	9950 2200 9950 2550
 $Comp
-L LED D?
+L Kurupira-Arthur-rescue:LED D?
 U 1 1 5B7B3797
 P 7600 750
@@
 $EndComp
 $Comp
-L R R?
+L Kurupira-Arthur-rescue:R R?
 U 1 1 5B7B37F2
 P 7900 750
@@
 Connection ~ 7400 1500
 $Comp
-L POT RV?
+L Kurupira-Arthur-rescue:POT RV?
 U 1 1 5B871DE1
 P 1350 6000
@@
 $EndComp
 $Comp
-L GND #PWR?
+L power:GND #PWR?
 U 1 1 5B871F49
 P 2450 6000
@@
 	2450 5950 2450 6000
 $Comp
-L BS108 Q?
+L Kurupira-Arthur-rescue:BS108 Q?
 U 1 1 5B873B34
 P 3350 5650
@@
 	3150 5650 2850 5650
 $Comp
-L +5V #PWR?
+L power:+5V #PWR?
 U 1 1 5B873F93
 P 3450 5450
@@
 	1200 6350 1200 4650
 $Comp
-L LM324 U?
+L Kurupira-Arthur-rescue:LM324 U?
 U 1 1 5B871BB5
 P 2550 5650
@@
 $EndComp
 $Comp
-L +5V #PWR?
+L power:+5V #PWR?
 U 1 1 5B87FDB9
 P 2100 5200
@@
 	2450 5200 2450 5350
 Wire Wire Line
-	1350 5200 2450 5200
+	1350 5200 2100 5200
 Wire Wire Line
 	1350 5200 1350 5850
@@
 	2100 6150 2100 5950
 Wire Wire Line
-	1750 5950 2450 5950
+	1750 5950 2100 5950
 Connection ~ 2450 5950
 Wire Wire Line
@@
 	2100 5550 2250 5550
 $Comp
-L R R?
+L Kurupira-Arthur-rescue:R R?
 U 1 1 5B880120
 P 1850 5400
@@
 $EndComp
 $Comp
-L R R?
+L Kurupira-Arthur-rescue:R R?
 U 1 1 5B8801A9
 P 1750 5800
@@
 $EndComp
 Wire Wire Line
-	1850 5550 1850 5650
+	1850 5550 1850 5600
 Wire Wire Line
 	1850 5650 1750 5650
@@
 Connection ~ 2100 5950
 $Comp
-L GND #PWR?
+L power:GND #PWR?
 U 1 1 5B88215A
 P 5600 5150
@@
 Wire Wire Line
 	5600 4850 5600 5150
+Wire Wire Line
+	9050 2600 9050 2700
+Wire Wire Line
+	7300 1150 7300 1500
+Wire Wire Line
+	8650 4600 8650 4700
+Wire Wire Line
+	10050 1950 10050 2000
+Wire Wire Line
+	7450 1150 7900 1150
+Wire Wire Line
+	2100 5200 2450 5200
+Wire Wire Line
+	1850 5600 1850 5650
+Wire Wire Line
+	2100 5950 2450 5950
 $EndSCHEMATC

Commit message: teste
Parts:
- removed Q?: BS108, TO_SOT_Packages_THT:TO-92_Molded_Narrow, symbol Kurupira-Arthur-rescue:BS108
- removed R? (x2): R, symbol Kurupira-Arthur-rescue:R
- removed RV?: POT, symbol Kurupira-Arthur-rescue:POT
- removed U?: FC-37, symbol Kurupira-Arthur-rescue:FC-37
- removed U?: LM324, symbol Kurupira-Arthur-rescue:LM324
- added U1: FC-37, symbol Kurupira-Arthur-rescue:FC-37
- gave numbers to parts that had none: 13
Connections:
- net +5V: now also J1.4 (5V)
- net GND: now also J1.14 (GND), J1.20 (GND), J1.25 (GND), J1.30 (GND), J1.34 (GND), J1.6 (GND), J1.9 (GND)
- net at U3.5 (Sensor): now also U1.1 (Sensor)
- net at U3.6 (Sensor): now also U1.2 (Sensor)
Other:
- note removed: "Parte que desliga a raspberry depois de uma tensão."
- moved on the sheet: Q1, R3, R4
