File: Kurupira 2.kicad_pcb (KiCad board)
At the start: 2 copper layers, 19.8 x 23.1 mm, 7 parts, among them J1 Conn_01x01_Female, J2 Conn_02x10_Odd_Even, J3 Conn_01x01_Female, J4 Conn_01x01_Female, Q1 Q_NPN_BEC

Commit message: Gerber files + Coppercam pcb
Adicionando os arquivos
Other:
- net class Default: clearance 0.5 -> 0.2
- rule trace_clearance: 0.5 -> 0.2
Changed lines of the file:
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@@
     (0 F.Cu signal)
     (31 B.Cu signal)
-    (32 B.Adhes user)
-    (33 F.Adhes user)
-    (34 B.Paste user)
-    (35 F.Paste user)
-    (36 B.SilkS user)
-    (37 F.SilkS user)
-    (38 B.Mask user)
-    (39 F.Mask user)
-    (40 Dwgs.User user)
-    (41 Cmts.User user)
-    (42 Eco1.User user)
-    (43 Eco2.User user)
+    (32 B.Adhes user hide)
+    (33 F.Adhes user hide)
+    (34 B.Paste user hide)
+    (35 F.Paste user hide)
+    (36 B.SilkS user hide)
+    (37 F.SilkS user hide)
+    (38 B.Mask user hide)
+    (39 F.Mask user hide)
+    (40 Dwgs.User user hide)
+    (41 Cmts.User user hide)
+    (42 Eco1.User user hide)
+    (43 Eco2.User user hide)
     (44 Edge.Cuts user)
-    (45 Margin user)
-    (46 B.CrtYd user)
-    (47 F.CrtYd user)
-    (48 B.Fab user)
-    (49 F.Fab user)
+    (45 Margin user hide)
+    (46 B.CrtYd user hide)
+    (47 F.CrtYd user hide)
+    (48 B.Fab user hide)
+    (49 F.Fab user hide)
   )
   (setup
     (last_trace_width 1)
-    (trace_clearance 0.5)
+    (trace_clearance 0.2)
     (zone_clearance 0.508)
     (zone_45_only no)
@@
     (mod_text_size 1 1)
     (mod_text_width 0.15)
-    (pad_size 1.5 1.5)
-    (pad_drill 0.6)
+    (pad_size 1.35 1.35)
+    (pad_drill 0.8)
     (pad_to_mask_clearance 0)
     (aux_axis_origin 0 0)
+    (grid_origin 176.784 108.458)
     (visible_elements 7FFFFFFF)
     (pcbplotparams
-      (layerselection 0x010fc_ffffffff)
+      (layerselection 0x01000_7fffffff)
       (usegerberextensions false)
       (usegerberattributes false)
       (usegerberadvancedattributes false)
-      (creategerberjobfile false)
+      (creategerberjobfile true)
       (excludeedgelayer true)
       (linewidth 0.100000)
@@
       (psnegative false)
       (psa4output false)
-      (plotreference true)
-      (plotvalue true)
+      (plotreference false)
+      (plotvalue false)
       (plotinvisibletext false)
       (padsonsilk false)
@@
       (drillshape 0)
       (scaleselection 1)
-      (outputdirectory ""))
+      (outputdirectory "Gerb/"))
   )
   (net 0 "")
@@
   (net 21 "Net-(J2-Pad6)")
   (net_class Default "This is the default net class."
-    (clearance 0.5)
+    (clearance 0.2)
     (trace_width 1)
     (via_dia 0.8)

Commit message: Mudando o pcb e as zonas
Parts:
- removed J4: Conn_01x01_Female, Pin_Headers:Pin_Header_Straight_1x01_Pitch2.00mm
Routing:
- net GND: track 0.00 -> 3.10 mm
Changed lines of the file:
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@@
     (thickness 1.6)
     (drawings 8)
-    (tracks 15)
+    (tracks 17)
     (zones 0)
-    (modules 7)
+    (modules 6)
     (nets 22)
   )
@@
     (mod_text_size 1 1)
     (mod_text_width 0.15)
-    (pad_size 1.35 1.35)
-    (pad_drill 0.8)
+    (pad_size 0.9 0.8)
+    (pad_drill 0)
     (pad_to_mask_clearance 0)
     (aux_axis_origin 0 0)
@@
     (add_net PIR)
     (add_net V_out)
-  )
-  (module Pin_Headers:Pin_Header_Straight_1x01_Pitch2.00mm (layer F.Cu)
-    (at 187.96 101.6)
-    (descr "Through hole straight pin header, 1x01, 2.00mm pitch, single row")
-    (tags "Through hole pin header THT 1x01 2.00mm single row")
-    (fp_text reference J1 (at 0 -2.06) (layer F.SilkS)
-      (effects (font (size 1 1) (thickness 0.15)))
-    )
-    (fp_text value Conn_01x01_Female (at 0 2.06) (layer F.Fab)
-      (effects (font (size 1 1) (thickness 0.15)))
-    )
-    (fp_text user %R (at 0 0 90) (layer F.Fab)
-      (effects (font (size 1 1) (thickness 0.15)))
-    )
-    (fp_line (start 1.5 -1.5) (end -1.5 -1.5) (layer F.CrtYd) (width 0.05))
-    (fp_line (start 1.5 1.5) (end 1.5 -1.5) (layer F.CrtYd) (width 0.05))
-    (fp_line (start -1.5 1.5) (end 1.5 1.5) (layer F.CrtYd) (width 0.05))
-    (fp_line (start -1.5 -1.5) (end -1.5 1.5) (layer F.CrtYd) (width 0.05))
-    (fp_line (start -1.06 -1.06) (end 0 -1.06) (layer F.SilkS) (width 0.12))
-    (fp_line (start -1.06 0) (end -1.06 -1.06) (layer F.SilkS) (width 0.12))
-    (fp_line (start -1.06 1) (end 1.06 1) (layer F.SilkS) (width 0.12))
-    (fp_line (start 1.06 1) (end 1.06 1.06) (layer F.SilkS) (width 0.12))
-    (fp_line (start -1.06 1) (end -1.06 1.06) (layer F.SilkS) (width 0.12))
-    (fp_line (start -1.06 1.06) (end 1.06 1.06) (layer F.SilkS) (width 0.12))
-    (fp_line (start -1 -0.5) (end -0.5 -1) (layer F.Fab) (width 0.1))
-    (fp_line (start -1 1) (end -1 -0.5) (layer F.Fab) (width 0.1))
-    (fp_line (start 1 1) (end -1 1) (layer F.Fab) (width 0.1))
-    (fp_line (start 1 -1) (end 1 1) (layer F.Fab) (width 0.1))
-    (fp_line (start -0.5 -1) (end 1 -1) (layer F.Fab) (width 0.1))
-    (pad 1 thru_hole rect (at 0 0) (size 1.35 1.35) (drill 0.8) (layers *.Cu *.Mask)
-      (net 2 PIR))
-    (model ${KISYS3DMOD}/Pin_Headers.3dshapes/Pin_Header_Straight_1x01_Pitch2.00mm.wrl
-      (at (xyz 0 0 0))
-      (scale (xyz 1 1 1))
-      (rotate (xyz 0 0 0))
-    )
   )
   (module Pin_Headers:Pin_Header_Straight_2x10_Pitch2.00mm (layer F.Cu)
@@
   )
   (module Pin_Headers:Pin_Header_Straight_1x01_Pitch2.00mm (layer F.Cu)
+    (at 187.96 101.6)
+    (descr "Through hole straight pin header, 1x01, 2.00mm pitch, single row")
+    (tags "Through hole pin header THT 1x01 2.00mm single row")
+    (fp_text reference J1 (at 0 -2.06) (layer F.SilkS)
+      (effects (font (size 1 1) (thickness 0.15)))
+    )
+    (fp_text value Conn_01x01_Female (at 0 2.06) (layer F.Fab)
+      (effects (font (size 1 1) (thickness 0.15)))
+    )
+    (fp_text user %R (at 0 0 90) (layer F.Fab)
+      (effects (font (size 1 1) (thickness 0.15)))
+    )
+    (fp_line (start 1.5 -1.5) (end -1.5 -1.5) (layer F.CrtYd) (width 0.05))
+    (fp_line (start 1.5 1.5) (end 1.5 -1.5) (layer F.CrtYd) (width 0.05))
+    (fp_line (start -1.5 1.5) (end 1.5 1.5) (layer F.CrtYd) (width 0.05))
+    (fp_line (start -1.5 -1.5) (end -1.5 1.5) (layer F.CrtYd) (width 0.05))
+    (fp_line (start -1.06 -1.06) (end 0 -1.06) (layer F.SilkS) (width 0.12))
+    (fp_line (start -1.06 0) (end -1.06 -1.06) (layer F.SilkS) (width 0.12))
+    (fp_line (start -1.06 1) (end 1.06 1) (layer F.SilkS) (width 0.12))
+    (fp_line (start 1.06 1) (end 1.06 1.06) (layer F.SilkS) (width 0.12))
+    (fp_line (start -1.06 1) (end -1.06 1.06) (layer F.SilkS) (width 0.12))
+    (fp_line (start -1.06 1.06) (end 1.06 1.06) (layer F.SilkS) (width 0.12))
+    (fp_line (start -1 -0.5) (end -0.5 -1) (layer F.Fab) (width 0.1))
+    (fp_line (start -1 1) (end -1 -0.5) (layer F.Fab) (width 0.1))
+    (fp_line (start 1 1) (end -1 1) (layer F.Fab) (width 0.1))
+    (fp_line (start 1 -1) (end 1 1) (layer F.Fab) (width 0.1))
+    (fp_line (start -0.5 -1) (end 1 -1) (layer F.Fab) (width 0.1))
+    (pad 1 thru_hole rect (at 0 0) (size 1.35 1.35) (drill 0.8) (layers *.Cu *.Mask)
+      (net 2 PIR))
+    (model ${KISYS3DMOD}/Pin_Headers.3dshapes/Pin_Header_Straight_1x01_Pitch2.00mm.wrl
+      (at (xyz 0 0 0))
+      (scale (xyz 1 1 1))
+      (rotate (xyz 0 0 0))
+    )
+  )
+  (module Pin_Headers:Pin_Header_Straight_1x01_Pitch2.00mm (layer F.Cu)
     (at 187.96 88.9)
     (descr "Through hole straight pin header, 1x01, 2.00mm pitch, single row")
@@
     )
   )
-  (module Pin_Headers:Pin_Header_Straight_1x01_Pitch2.00mm (layer F.Cu)
-    (at 187.96 97.028)
-    (descr "Through hole straight pin header, 1x01, 2.00mm pitch, single row")
-    (tags "Through hole pin header THT 1x01 2.00mm single row")
-    (fp_text reference J4 (at 0 -2.06) (layer F.SilkS)
-      (effects (font (size 1 1) (thickness 0.15)))
-    )
-    (fp_text value Conn_01x01_Female (at 0 2.06) (layer F.Fab)
-      (effects (font (size 1 1) (thickness 0.15)))
-    )
-    (fp_text user %R (at 0 0 90) (layer F.Fab)
-      (effects (font (size 1 1) (thickness 0.15)))
-    )
-    (fp_line (start 1.5 -1.5) (end -1.5 -1.5) (layer F.CrtYd) (width 0.05))
-    (fp_line (start 1.5 1.5) (end 1.5 -1.5) (layer F.CrtYd) (width 0.05))
-    (fp_line (start -1.5 1.5) (end 1.5 1.5) (layer F.CrtYd) (width 0.05))
-    (fp_line (start -1.5 -1.5) (end -1.5 1.5) (layer F.CrtYd) (width 0.05))
-    (fp_line (start -1.06 -1.06) (end 0 -1.06) (layer F.SilkS) (width 0.12))
-    (fp_line (start -1.06 0) (end -1.06 -1.06) (layer F.SilkS) (width 0.12))
-    (fp_line (start -1.06 1) (end 1.06 1) (layer F.SilkS) (width 0.12))
-    (fp_line (start 1.06 1) (end 1.06 1.06) (layer F.SilkS) (width 0.12))
-    (fp_line (start -1.06 1) (end -1.06 1.06) (layer F.SilkS) (width 0.12))
-    (fp_line (start -1.06 1.06) (end 1.06 1.06) (layer F.SilkS) (width 0.12))
-    (fp_line (start -1 -0.5) (end -0.5 -1) (layer F.Fab) (width 0.1))
-    (fp_line (start -1 1) (end -1 -0.5) (layer F.Fab) (width 0.1))
-    (fp_line (start 1 1) (end -1 1) (layer F.Fab) (width 0.1))
-    (fp_line (start 1 -1) (end 1 1) (layer F.Fab) (width 0.1))
-    (fp_line (start -0.5 -1) (end 1 -1) (layer F.Fab) (width 0.1))
-    (pad 1 thru_hole rect (at 0 0) (size 1.35 1.35) (drill 0.8) (layers *.Cu *.Mask)
-      (net 1 GND))
-    (model ${KISYS3DMOD}/Pin_Headers.3dshapes/Pin_Header_Straight_1x01_Pitch2.00mm.wrl
-      (at (xyz 0 0 0))
-      (scale (xyz 1 1 1))
-      (rotate (xyz 0 0 0))
-    )
-  )
   (module TO_SOT_Packages_SMD:SOT-23 (layer F.Cu)
     (at 180.848 93.98 90)
@@
       (net 15 V_out))
     (pad 2 smd rect (at -1 0.95 90) (size 0.9 0.8) (layers F.Cu F.Paste F.Mask)
-      (net 1 GND))
+      (net 1 GND) (zone_connect 2))
     (pad 1 smd rect (at -1 -0.95 90) (size 0.9 0.8) (layers F.Cu F.Paste F.Mask)
       (net 19 "Net-(Q1-Pad1)"))
@@
   (gr_line (start 176.784 108.458) (end 196.596 108.458) (angle 90) (layer Edge.Cuts) (width 0.1))
   (gr_line (start 196.596 85.344) (end 176.784 85.344) (angle 90) (layer Edge.Cuts) (width 0.1))
+  (segment (start 193.04 96.9) (end 190.118 96.9) (width 1) (layer F.Cu) (net 1) (status 400000))
+  (segment (start 190.118 96.9) (end 189.992 96.774) (width 1) (layer F.Cu) (net 1))
   (segment (start 183.864 101.6) (end 187.96 101.6) (width 1) (layer F.Cu) (net 2) (status C00000))
-  (segment (start 187.96 101.6) (end 190.34 101.6) (width 1) (layer F.Cu) (net 2) (status 400000))
-  (segment (start 190.34 101.6) (end 193.04 98.9) (width 1) (layer F.Cu) (net 2) (status 800000))
+  (segment (start 193.04 98.9) (end 190.66 98.9) (width 1) (layer F.Cu) (net 2) (status 400000))
+  (segment (start 190.66 98.9) (end 187.96 101.6) (width 1) (layer F.Cu) (net 2) (status 800000))
   (segment (start 193.04 92.9) (end 180.928 92.9) (width 1) (layer F.Cu) (net 15) (status C00000))
   (segment (start 180.928 92.9) (end 180.848 92.98) (width 1) (layer F.Cu) (net 15) (status C00000))
@@
   (segment (start 194.31 86.36) (end 190.5 86.36) (width 1) (layer F.Cu) (net 16))
   (segment (start 195.04 87.09) (end 194.31 86.36) (width 1) (layer F.Cu) (net 16))
-  (segment (start 179.864 101.6) (end 179.864 94.964) (width 1) (layer F.Cu) (net 19) (status C00000))
   (segment (start 179.864 94.964) (end 179.88 94.98) (width 1) (layer F.Cu) (net 19) (status C00000))
   (segment (start 179.88 94.98) (end 179.898 94.98) (width 1) (layer F.Cu) (net 19) (status C00000))
+  (segment (start 179.864 101.6) (end 179.864 94.964) (width 1) (layer F.Cu) (net 19) (status C00000))
+  (zone (net 0) (net_name "") (layer F.Cu) (hatch edge 0.508)
+    (connect_pads (clearance 0.508))
+    (min_thickness 0.254)
+    (keepout (tracks not_allowed) (vias not_allowed) (copperpour not_allowed))
+    (fill (arc_segments 16) (thermal_gap 0.508) (thermal_bridge_width 0.508))
+    (polygon
+      (pts
+        (xy 194.056 95.758) (xy 191.516 95.758) (xy 191.516 87.63) (xy 196.088 87.63) (xy 196.088 107.95)
+        (xy 191.516 107.95) (xy 191.516 98.298) (xy 194.056 98.298)
+      )
+    )
+  )
   (zone (net 1) (net_name GND) (layer F.Cu) (hatch edge 0.508)
     (connect_pads (clearance 0.508))
@@
     (polygon
       (pts
-        (xy 177.8 86.36) (xy 177.8 107.315) (xy 195.58 107.315) (xy 196.215 86.36)
+        (xy 181.356 94.234) (xy 181.356 99.822) (xy 191.008 99.822) (xy 191.008 94.234)
       )
     )
